File: 2206Q/riscduino_board/Riscduino_Uno_Rev1.0/Riscduino_Uno.kicad_sch (KiCad schematic)
At the start: 79 parts, among them J1 USB_B_Micro, J10 Conn_01x01, J11 Conn_01x01, J2 ISP, J3 Conn_01x08_Pin, J4 Conn_01x06_Pin, J5 Conn_01x08_Pin, J6 Conn_01x10_Pin, J7 Conn_02x04_Odd_Even, J8 Conn_01x01, J9 Conn_01x01, SW1 4Pin Round Button SPST Straig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, U1 LM1117S-ADJ, U2 LM1117MP-3.3, U3 Riscduino, U4 CP2102N-Axx-xQFN28, U5 W25Q32JVSS, U6 W25Q32JVSS, U7 23LC1024-I/P, U8 MAX1232ESA+T, X1 ASE-10.000MHZ-LC-T

Commit message: 1.0.3 Update
Parts:
- removed C19: 0.1uf, Capacitor_SMD:C_0603_1608Metric_Pad1.08x0.95mm_HandSolder, symbol Library:C
- removed C22: 0.1uF, Capacitor_SMD:C_0603_1608Metric_Pad1.08x0.95mm_HandSolder, symbol Device:C
- removed JP1: Jumper_2_Open, Connector_PinHeader_2.54mm:PinHeader_1x02_P2.54mm_Vertical, symbol Jumper:Jumper_2_Open
- removed JP3: Jumper_2, Connector_PinHeader_2.54mm:PinHeader_1x02_P2.54mm_Vertical, symbol Jumper:Jumper_2_Bridged
- removed U4: CP2102N-Axx-xQFN28, Package_DFN_QFN:QFN-28-1EP_5x5mm_P0.5mm_EP3.35x3.35mm, symbol Interface_USB:CP2102N-Axx-xQFN28
- removed U5: W25Q32JVSS, Package_SO:SOIC-8_5.23x5.23mm_P1.27mm, symbol Memory_Flash:W25Q32JVSS
- removed U8: MAX1232ESA+T, MAX1232ESA+T:SOIC127P600X175-8N, symbol MAX1232ESA+T:MAX1232ESA+T
- added C19: 0.1uF, Capacitor_SMD:C_0603_1608Metric_Pad1.08x0.95mm_HandSolder, symbol Device:C
- added C22: 0.1uf, Capacitor_SMD:C_0603_1608Metric_Pad1.08x0.95mm_HandSolder, symbol Library:C
- added H1, H2, H3, H4: MountingHole, MountingHole:MountingHole_3.2mm_M3, symbol Mechanical:MountingHole
- added JP1: Jumper_2, Connector_PinHeader_2.54mm:PinHeader_1x02_P2.54mm_Vertical, symbol Jumper:Jumper_2_Bridged
- added R23, R24, R25, R26: 10K, Resistor_SMD:R_0603_1608Metric_Pad0.98x0.95mm_HandSolder, symbol Device:R
- added R27, R28, R29, R30, R31, R32: 470 Ohm, Resistor_SMD:R_0603_1608Metric_Pad0.98x0.95mm_HandSolder, symbol Device:R
- added TP1: TestPoint, Connector_PinHeader_2.54mm:PinHeader_1x01_P2.54mm_Vertical, symbol Connector:TestPoint
- added U4: CH340C, Package_SO:SOIC-16_3.9x9.9mm_P1.27mm, symbol Interface_USB:CH340C
- added U5: MAX1232ESA+T, Package_SO:SOIC-8-1EP_3.9x4.9mm_P1.27mm_EP2.29x3mm, symbol MAX1232ESA+T:MAX1232ESA+T
- added U8: 23LC1024-I/P, Package_DIP:DIP-8_W7.62mm_LongPads, symbol Memory_Flash:W25Q32JVSS
- C1: footprint Capacitor_SMD:C_0805_2012Metric_Pad1.18x1.45mm_HandSolder -> Button_Switch_SMD:SW_SPST_CK_KXT3
- C11: value 0.1uF -> 22uF; footprint Capacitor_SMD:C_0603_1608Metric_Pad1.08x0.95mm_HandSolder -> Capacitor_SMD:C_0805_2012Metric_Pad1.18x1.45mm_HandSolder
- C12: value 22uF -> 0.1uF; footprint Capacitor_SMD:C_0805_2012Metric_Pad1.18x1.45mm_HandSolder -> Capacitor_SMD:C_0603_1608Metric_Pad1.08x0.95mm_HandSolder
- D1: value RED LED -> BLUE LED
- D3: value BLUE LED -> RED LED
- R1: value 470 Ohm -> DNI
- R10, R9: value 470 Ohm -> 0E
- R11, R2, R3, R4, R8: value 10K -> 0E
- R19, R20, R21, R22: value 470 Ohm -> 10K
- R5, R6: value 10K -> DNI
- R7: value 10K -> 470 Ohm
- SW1: footprint Switch_E-Switch_TL3315NF250Q:E-Switch-TL3315NF250Q-0-0-0 -> Button_Switch_SMD:SW_Push_SPST_NO_Alps_SKRK
- U3: footprint Package_DFN_QFN:QFN-64-1EP_9x9mm_P0.5mm_EP7.65x7.65mm -> Package_DFN_QFN:RISCDUINO_QFN-64-1EP_9x9mm_P0.5mm_EP7.65x7.65mm_NEW
- U7: value 23LC1024-I/P -> W25Q32JVSS; footprint Package_DIP:DIP-8_W7.62mm_LongPads -> Package_SO:SOIC-8_5.23x5.23mm_P1.27mm
- X1: footprint Oscillator:Oscillator_SMD_Abracon_ASE-4Pin_3.2x2.5mm_HandSoldering -> Crystal:Crystal_SMD_Abracon_ABM8G-4Pin_3.2x2.5mm
Connections:
- net +1V8: now also R3.1, R4.1, R7.1, R9.2, JP1.1 (A), JP1.2 (B); no longer C21.2, C5.2, C6.2, JP2.1 (A), JP2.2 (B), R1.1, U3.18 (vccd), U3.49 (vccd1), U3.63 (vccd2)
- net +3.3V: now also C16.1, C18.1, C20.2, C21.1, JP2.2 (B), R19.1, R20.1, R21.1, R22.1, R8.2, R23.1, R24.1, R25.1, R26.1, R27.2, R28.2, R29.2, R30.2, R31.2, R32.2, U4.16 (VCC), U5.2 (TD), U5.8 (VCC), U8.8 (VCC); no longer C20.1, R10.2, R11.1, R19.2, R20.2, R21.2, R22.2, R3.1, R4.1, R5.1, R6.1, R7.1, R8.1, R9.2
- net +3.3VP: now also C7.1, JP2.1 (A), R2.1, R5.1; no longer C8.1
- net +5V: now also C8.1, R1.1; no longer C1.1, C16.1, C18.1, C3.1, C7.1, R2.1, U1.3 (VI)
- net CARAVEL_FLASH_IO0: now also R18.2, U6.5 (DI(IO0)); no longer R11.2
- net CARAVEL_FLASH_IO1: now also R16.2, U6.2 (DO(IO1)); no longer R7.2
- net CARAVEL_FLASH_IO2: now also R14.2, U6.3 (IO2); no longer R5.2
- net CARAVEL_FLASH_IO3: now also R12.2, U6.7 (IO3); no longer R3.2
- net CARAVEL_FLASH_SCK: now also R20.2, U6.6 (CLK); no longer R13.2
- net CARAVEL_FLASH_SSN: now also R22.2, U6.1 (~{CS}); no longer R15.2
- net GND: now also C20.1, C21.2, C5.2, D3.1 (K), R6.2, C19.1, C22.1, U4.1 (GND), U5.3 (TOL), U5.4 (GND), U8.4 (GND); no longer C20.2, C21.1, C5.1, D1.1 (K)
- net USB_D+: now also U4.5 (UD+)
- net USB_D-: now also U4.6 (UD-)
- net USER_FLASH_IO0: now also R19.2, U8.5 (DI(IO0)); no longer R12.2, U6.5 (DI(IO0))
- net USER_FLASH_IO1: now also R17.2, U8.2 (DO(IO1)); no longer R8.2, U6.2 (DO(IO1))
- net USER_FLASH_IO2: now also R15.2, U8.3 (IO2); no longer R6.2, U6.3 (IO2)
- net USER_FLASH_IO3: now also R13.2, U8.7 (IO3); no longer R4.2, U6.7 (IO3)
- net USER_FLASH_SCK: now also R21.2, U8.6 (CLK); no longer R14.2, U6.6 (CLK)
- net USER_FLASH_SSN: now also U7.1 (~{CS}), R23.2; no longer R16.2, U6.1 (~{CS})
- net USER_SRAM_SSN: now also R24.2, U8.1 (~{CS}); no longer R17.2, U7.1 (~{CS})
- net ardunio_d0: now also D1.1 (K), R10.2; no longer D3.1 (K)
- net ardunio_d1: now also D2.1 (K), R11.2; no longer D4.1 (K)
- net ardunio_d2: now also D4.1 (K); no longer D5.1 (K)
- net gpio: now also D5.1 (K); no longer D2.1 (K)
- net ~{RST}: now also R26.2, U5.6 (~{RST})
- net at D4.2 (A): now also R31.1; no longer R20.1
- net at RV1.2, U1.1 (ADJ): now also R7.2, RV1.1; no longer R1.2
- net at R2.2: now also C1.1, C3.1, R1.2, U1.3 (VI)
- net at X1.1 (EN): now also R5.2, R6.1
- net at D6.2 (A): now also R32.1; no longer R22.1
- net at R10.1: now also U4.2 (TXD); no longer D2.2 (A)
- net at SW1.2: now also U5.1 (~{PB_RST})
- net at D3.2 (A): now also R27.1; no longer R19.1
- net at D5.2 (A): now also R28.1; no longer R21.1
- net at D1.2 (A): now also R29.1; no longer R9.1
- new net: TP1.1, U4.13 (~{DTR})
- new net: R11.1, U4.3 (RXD)
- new net: C19.2, R8.1, U4.4 (V3)
- new net: D2.2 (A), R30.1
- new net: R25.2, U5.7 (~{ST})
- new net vccd0: C22.2, R9.1, U3.18 (vccd)
- new net vccd1: C6.2, R4.2, U3.49 (vccd1)
- new net vccd2: C5.1, R3.2, U3.63 (vccd2)

Commit message: 1.0.4
Connections:
- net +1V8: no longer C10.1, C13.1, JP1.1 (A), R7.1, U1.2 (VO)
- net +3.3V: now also C12.1, R5.1, X1.4 (Vdd)
- net +3.3VP: no longer C12.1, R5.1, X1.4 (Vdd)
- new net +1.8VP: C10.1, C13.1, JP1.1 (A), R7.1, U1.2 (VO)
Changed lines of the file:
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@@
   (junction (at 347.726 37.084) (diameter 0) (color 0 0 0 0)
   )
-  (junction (at 80.264 252.73) (diameter 0) (color 0 0 0 0)
+  (junction (at 81.28 373.38) (diameter 0) (color 0 0 0 0)
   )
   (junction (at 71.374 262.89) (diameter 0) (color 0 0 0 0)
@@
   (junction (at 323.85 62.738) (diameter 0) (color 0 0 0 0)
   )
-  (junction (at 81.28 373.38) (diameter 0) (color 0 0 0 0)
+  (junction (at 75.184 371.856) (diameter 0) (color 0 0 0 0)
   )
   (junction (at 320.548 201.422) (diameter 0) (color 0 0 0 0)
@@
   (junction (at 343.916 330.708) (diameter 0) (color 0 0 0 0)
   )
-  (junction (at 86.614 206.248) (diameter 0) (color 0 0 0 0)
-  )
   (junction (at 318.77 67.818) (diameter 0) (color 0 0 0 0)
   )
@@
     (stroke (width 0) (type default))
   )
-  (wire (pts (xy 80.264 250.19) (xy 80.264 252.73))
-    (stroke (width 0) (type default))
-  )
   (wire (pts (xy 47.498 206.248) (xy 51.816 206.248))
     (stroke (width 0) (type default))
@@
     (stroke (width 0) (type default))
   )
-  (wire (pts (xy 86.614 202.184) (xy 86.614 206.248))
-    (stroke (width 0) (type default))
-  )
   (wire (pts (xy 370.84 320.294) (xy 375.412 320.294))
     (stroke (width 0) (type default))
@@
     (stroke (width 0) (type default))
   )
+  (wire (pts (xy 81.28 371.856) (xy 81.28 373.38))
+    (stroke (width 0) (type default))
+  )
   (wire (pts (xy 507.238 318.77) (xy 508.762 318.77))
     (stroke (width 0) (type default))
@@
     (stroke (width 0) (type default))
   )
-  (wire (pts (xy 86.614 206.248) (xy 89.408 206.248))
-    (stroke (width 0) (type default))
-  )
   (wire (pts (xy 170.942 274.32) (xy 171.45 274.32))
     (stroke (width 0) (type default))
@@
     (stroke (width 0) (type default))
   )
-  (wire (pts (xy 81.28 370.84) (xy 81.28 373.38))
-    (stroke (width 0) (type default))
-  )
-  (wire (pts (xy 81.28 373.38) (xy 81.28 375.92))
-    (stroke (width 0) (type default))
-  )
   (wire (pts (xy 62.23 260.35) (xy 62.23 262.89))
     (stroke (width 0) (type default))
@@
     (stroke (width 0) (type default))
   )
-  (wire (pts (xy 81.28 373.38) (xy 86.36 373.38))
-    (stroke (width 0) (type default))
-  )
   (wire (pts (xy 106.68 109.22) (xy 106.68 113.03))
     (stroke (width 0) (type default))
@@
     (stroke (width 0) (type default))
   )
+  (wire (pts (xy 81.28 373.38) (xy 81.28 375.92))
+    (stroke (width 0) (type default))
+  )
   (wire (pts (xy 329.692 358.902) (xy 329.692 358.648))
     (stroke (width 0) (type default))
@@
     (stroke (width 0) (type default))
   )
-  (wire (pts (xy 63.5 374.65) (xy 63.5 373.38))
-    (stroke (width 0) (type default))
-  )
   (wire (pts (xy 315.214 129.54) (xy 337.566 129.54))
     (stroke (width 0) (type default))
@@
     (stroke (width 0) (type default))
   )
+  (wire (pts (xy 63.5 371.856) (xy 75.184 371.856))
+    (stroke (width 0) (type default))
+  )
   (wire (pts (xy 376.428 376.428) (xy 383.032 376.428))
     (stroke (width 0) (type default))
@@
     (stroke (width 0) (type default))
   )
+  (wire (pts (xy 75.184 370.586) (xy 75.184 371.856))
+    (stroke (width 0) (type default))
+  )
   (wire (pts (xy 148.59 246.38) (xy 158.242 246.38))
     (stroke (width 0) (type default))
@@
     (stroke (width 0) (type default))
   )
-  (wire (pts (xy 80.264 252.73) (xy 84.328 252.73))
-    (stroke (width 0) (type default))
-  )
   (wire (pts (xy 80.01 81.28) (xy 86.36 81.28))
     (stroke (width 0) (type default))
@@
     (stroke (width 0) (type default))
   )
+  (wire (pts (xy 81.28 373.38) (xy 86.36 373.38))
+    (stroke (width 0) (type default))
+  )
   (wire (pts (xy 494.538 257.048) (xy 496.824 257.048))
     (stroke (width 0) (type default))
@@
     (stroke (width 0) (type default))
   )
+  (wire (pts (xy 75.184 371.856) (xy 81.28 371.856))
+    (stroke (width 0) (type default))
+  )
   (wire (pts (xy 326.898 353.822) (xy 330.454 353.822))
     (stroke (width 0) (type default))
@@
     (stroke (width 0) (type default))
   )
+  (wire (pts (xy 63.5 371.856) (xy 63.5 374.65))
+    (stroke (width 0) (type default))
+  )
   (wire (pts (xy 370.84 332.994) (xy 376.682 332.994))
     (stroke (width 0) (type default))
@@
     (stroke (width 0) (type default))
   )
-  (wire (pts (xy 80.01 206.248) (xy 86.614 206.248))
+  (wire (pts (xy 80.01 206.248) (xy 89.408 206.248))
     (stroke (width 0) (type default))
   )
@@
     (stroke (width 0) (type default))
   )
-  (wire (pts (xy 63.5 373.38) (xy 81.28 373.38))
-    (stroke (width 0) (type default))
-  )
   (wire (pts (xy 506.222 325.628) (xy 509.27 325.628))
     (stroke (width 0) (type default))
@@
     (stroke (width 0) (type default))
   )
-  (wire (pts (xy 71.374 252.73) (xy 80.264 252.73))
+  (wire (pts (xy 71.374 252.73) (xy 84.328 252.73))
     (stroke (width 0) (type default))
   )
@@
     (effects (font (size 1.27 1.27)) (justify left bottom))
   )
+  (label "+1.8VP" (at 72.898 252.73 0) (fields_autoplaced)
+    (effects (font (size 1.27 1.27)) (justify left bottom))
+  )
   (label "vccd2" (at 60.96 93.98 0) (fields_autoplaced)
     (effects (font (size 1.27 1.27)) (justify left bottom))
   )
+  (label "+3.3VP" (at 79.248 206.248 0) (fields_autoplaced)
+    (effects (font (size 1.27 1.27)) (justify left bottom))
+  )
   (global_label "USER_FLASH_SCK" (shape bidirectional) (at 395.224 51.562 180) (fields_autoplaced)
     (effects (font (size 1.27 1.27)) (justify right))
@@
     )
   )
-  (symbol (lib_id "power:+3.3VP") (at 81.28 370.84 0) (unit 1)
-    (in_bom yes) (on_board yes) (dnp no) (fields_autoplaced)
-    (property "Reference" "#PWR021" (at 85.09 372.11 0)
-      (effects (font (size 1.27 1.27)) hide)
-    )
-    (property "Value" "+3.3V" (at 81.28 366.776 0)
-      (effects (font (size 1.27 1.27)))
-    )
-    (property "Footprint" "" (at 81.28 370.84 0)
-      (effects (font (size 1.27 1.27)) hide)
-    )
-    (property "Datasheet" "" (at 81.28 370.84 0)
-      (effects (font (size 1.27 1.27)) hide)
-    )
-    (pin "1")
-    (instances
-      (project "Riscduino_Uno"
-        (path "/3385a618-de98-459b-bc8d-0b8733b3fac9"
-          (reference "#PWR021") (unit 1)
-        )
-      )
-    )
-  )
   (symbol (lib_id "Device:R") (at 323.088 183.388 0) (unit 1)
     (in_bom yes) (on_board yes) (dnp no)
@@
     )
   )
-  (symbol (lib_id "power:+3.3VP") (at 86.614 202.184 0) (unit 1)
-    (in_bom yes) (on_board yes) (dnp no) (fields_autoplaced)
-    (property "Reference" "#PWR025" (at 90.424 203.454 0)
-      (effects (font (size 1.27 1.27)) hide)
-    )
-    (property "Value" "+3.3VP" (at 86.614 198.882 0)
-      (effects (font (size 1.27 1.27)))
-    )
-    (property "Footprint" "" (at 86.614 202.184 0)
-      (effects (font (size 1.27 1.27)) hide)
-    )
-    (property "Datasheet" "" (at 86.614 202.184 0)
-      (effects (font (size 1.27 1.27)) hide)
-    )
-    (pin "1")
-    (instances
-      (project "Riscduino_Uno"
-        (path "/3385a618-de98-459b-bc8d-0b8733b3fac9"
-          (reference "#PWR025") (unit 1)
-        )
-      )
-    )
-  )
   (symbol (lib_id "Device:R") (at 334.01 114.046 0) (unit 1)
     (in_bom yes) (on_board yes) (dnp no)
@@
     )
   )
+  (symbol (lib_id "power:+3.3V") (at 75.184 370.586 0) (unit 1)
+    (in_bom yes) (on_board yes) (dnp no) (fields_autoplaced)
+    (property "Reference" "#PWR021" (at 75.184 374.396 0)
+      (effects (font (size 1.27 1.27)) hide)
+    )
+    (property "Value" "+3.3V" (at 75.184 366.776 0)
+      (effects (font (size 1.27 1.27)))
+    )
+    (property "Footprint" "" (at 75.184 370.586 0)
+      (effects (font (size 1.27 1.27)) hide)
+    )
+    (property "Datasheet" "" (at 75.184 370.586 0)
+      (effects (font (size 1.27 1.27)) hide)
+    )
+    (pin "1")
+    (instances
+      (project "Riscduino_Uno"
+        (path "/3385a618-de98-459b-bc8d-0b8733b3fac9"
+          (reference "#PWR021") (unit 1)
+        )
+      )
+    )
+  )
   (symbol (lib_id "Device:R") (at 63.5 391.16 0) (unit 1)
     (in_bom yes) (on_board yes) (dnp no)
@@
         )
       )
-    )
-  )
-  (symbol (lib_id "power:+1V8") (at 80.264 250.19 0) (unit 1)
-    (in_bom yes) (on_board yes) (dnp no) (fields_autoplaced)
-    (property "Reference" "#PWR020" (at 80.264 254 0)
-      (effects (font (size 1.27 1.27)) hide)
-    )
-    (property "Value" "+1.8VP" (at 80.264 246.38 0)
-      (effects (font (size 1.27 1.27)))
-    )
-    (property "Footprint" "" (at 80.264 250.19 0)
-      (effects (font (size 1.27 1.27)) hide)
-    )
-    (property "Datasheet" "" (at 80.264 250.19 0)
-      (effects (font (size 1.27 1.27)) hide)
-    )
-    (pin "1")
-    (instances
-      (project "Riscduino_Uno"
-        (path "/3385a618-de98-459b-bc8d-0b8733b3fac9"
-          (reference "#PWR020") (unit 1)
-        )
-      )

Commit message: 1.0.7 DRC Clean, Power Routed
Parts:
- SW1: footprint Button_Switch_SMD:SW_Push_SPST_NO_Alps_SKRK -> Riscduino.Library:SW_SPST_EVPBF_TS4550TP
- U3: footprint Package_DFN_QFN:RISCDUINO_QFN-64-1EP_9x9mm_P0.5mm_EP7.65x7.65mm_NEW -> Riscduino.Library:RISCDUINO_QFN-64-1EP_9x9mm_P0.5mm_EP7.65x7.65mm_NEW
Connections:
- net +3.3V: now also J2.2 (Pin_2)
- net +3.3VP: no longer J2.2 (Pin_2)
Changed lines of the file:
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@@
     (stroke (width 0) (type default))
   )
+  (wire (pts (xy 182.88 378.46) (xy 185.674 378.46))
+    (stroke (width 0) (type default))
+  )
   (wire (pts (xy 64.516 327.152) (xy 64.516 329.184))
     (stroke (width 0) (type default))
@@
     (stroke (width 0) (type default))
   )
+  (wire (pts (xy 185.674 378.46) (xy 185.674 376.936))
+    (stroke (width 0) (type default))
+  )
   (wire (pts (xy 329.946 377.952) (xy 334.772 377.952))
     (stroke (width 0) (type default))
@@
     (stroke (width 0) (type default))
   )
-  (wire (pts (xy 186.69 378.46) (xy 186.69 375.92))
-    (stroke (width 0) (type default))
-  )
   (wire (pts (xy 186.69 383.54) (xy 186.69 384.556))
     (stroke (width 0) (type default))
@@
     (stroke (width 0) (type default))
   )
-  (wire (pts (xy 182.88 378.46) (xy 186.69 378.46))
-    (stroke (width 0) (type default))
-  )
   (wire (pts (xy 189.23 91.44) (xy 189.23 93.98))
     (stroke (width 0) (type default))
@@
     )
   )
-  (symbol (lib_id "power:+3.3VP") (at 186.69 375.92 0) (unit 1)
-    (in_bom yes) (on_board yes) (dnp no) (fields_autoplaced)
-    (property "Reference" "#PWR052" (at 190.5 377.19 0)
-      (effects (font (size 1.27 1.27)) hide)
-    )
-    (property "Value" "+3.3V" (at 186.69 371.856 0)
-      (effects (font (size 1.27 1.27)))
-    )
-    (property "Footprint" "" (at 186.69 375.92 0)
-      (effects (font (size 1.27 1.27)) hide)
-    )
-    (property "Datasheet" "" (at 186.69 375.92 0)
-      (effects (font (size 1.27 1.27)) hide)
-    )
-    (pin "1")
-    (instances
-      (project "Riscduino_Uno"
-        (path "/3385a618-de98-459b-bc8d-0b8733b3fac9"
-          (reference "#PWR052") (unit 1)
-        )
-      )
-    )
-  )
   (symbol (lib_id "power:GND") (at 99.06 113.03 0) (unit 1)
     (in_bom yes) (on_board yes) (dnp no)
@@
       (effects (font (size 1.27 1.27)) (justify left))
     )
-    (property "Footprint" "Package_DFN_QFN:RISCDUINO_QFN-64-1EP_9x9mm_P0.5mm_EP7.65x7.65mm_NEW" (at 129.54 80.01 0)
+    (property "Footprint" "Riscduino.Library:RISCDUINO_QFN-64-1EP_9x9mm_P0.5mm_EP7.65x7.65mm_NEW" (at 129.54 80.01 0)
       (effects (font (size 1.27 1.27)) hide)
     )
@@
     )
   )
+  (symbol (lib_id "power:+3.3V") (at 185.674 376.936 0) (unit 1)
+    (in_bom yes) (on_board yes) (dnp no) (fields_autoplaced)
+    (property "Reference" "#PWR020" (at 185.674 380.746 0)
+      (effects (font (size 1.27 1.27)) hide)
+    )
+    (property "Value" "+3.3V" (at 185.674 373.38 0)
+      (effects (font (size 1.27 1.27)))
+    )
+    (property "Footprint" "" (at 185.674 376.936 0)
+      (effects (font (size 1.27 1.27)) hide)
+    )
+    (property "Datasheet" "" (at 185.674 376.936 0)
+      (effects (font (size 1.27 1.27)) hide)
+    )
+    (pin "1")
+    (instances
+      (project "Riscduino_Uno"
+        (path "/3385a618-de98-459b-bc8d-0b8733b3fac9"
+          (reference "#PWR020") (unit 1)
+        )
+      )
+    )
+  )
   (symbol (lib_id "Device:R") (at 63.5 378.46 0) (unit 1)
     (in_bom yes) (on_board yes) (dnp no)
@@
       (effects (font (size 1.27 1.27)) hide)
     )
-    (property "Footprint" "Button_Switch_SMD:SW_Push_SPST_NO_Alps_SKRK" (at 318.77 257.81 0)
+    (property "Footprint" "Riscduino.Library:SW_SPST_EVPBF_TS4550TP" (at 318.77 257.81 0)
       (effects (font (size 1.27 1.27)) hide)
     )

Commit message: Gerber 1.0 Release to Lion Circuit
Parts:
- renumbered C25 to C1, C6 to C10, C15 to C11, C21 to C12, C9 to C13, C11 to C14, C1 to C15, C7 to C16, C16 to C17, C10 to C18, C24 to C19, C26 to C2, C2 to C20, C8 to C21, C13 to C22, C3 to C23, C4 to C24, C18 to C25, C19 to C26, C12 to C3, C23 to C4, C14 to C6, C22 to C7, C17 to C8, C20 to C9, D6 to D1, D4 to D2, D5 to D3, D3 to D4, D2 to D5, D1 to D6, H3 to H1, H4 to H3, H1 to H4, J3 to J1, J1 to J10, J6 to J11, J4 to J2, J8 to J3, J7 to J4, J2 to J5, J11 to J6, J9 to J7, J10 to J8, J5 to J9, JP2 to JP1, JP1 to JP2, R26 to R1, R2 to R10, R10 to R11, R1 to R12, R9 to R13, R7 to R14, R30 to R15, R29 to R16, R11 to R17, R5 to R18, R6 to R19, R25 to R2, R32 to R20, R31 to R21, R24 to R22, R27 to R23, R28 to R24, R17 to R25, R23 to R26, R18 to R27, R22 to R28, R20 to R29, R13 to R3, R19 to R30, R21 to R31, R8 to R32, R16 to R4, R14 to R5, R15 to R6, R12 to R7, R4 to R8, R3 to R9, U5 to U1, U6 to U2, U7 to U3, U8 to U4, U3 to U5, U2 to U6, U1 to U7, U4 to U8

Commit message: 1.0.9
Connections:
- net GND: now also J10.6 (Shield)
Changed lines of the file:
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@@
   (junction (at 81.28 397.51) (diameter 0) (color 0 0 0 0)
   )
+  (junction (at 64.516 328.168) (diameter 0) (color 0 0 0 0)
+  )
   (junction (at 347.726 103.886) (diameter 0) (color 0 0 0 0)
   )
@@
     (stroke (width 0) (type default))
   )
+  (wire (pts (xy 61.976 328.168) (xy 64.516 328.168))
+    (stroke (width 0) (type default))
+  )
   (wire (pts (xy 116.84 109.22) (xy 116.84 114.3))
     (stroke (width 0) (type default))
@@
     (stroke (width 0) (type default))
   )
+  (wire (pts (xy 64.516 328.168) (xy 64.516 329.184))
+    (stroke (width 0) (type default))
+  )
   (wire (pts (xy 314.452 198.882) (xy 323.088 198.882))
     (stroke (width 0) (type default))
@@
     (stroke (width 0) (type default))
   )
-  (wire (pts (xy 64.516 327.152) (xy 64.516 329.184))
+  (wire (pts (xy 64.516 327.152) (xy 64.516 328.168))
     (stroke (width 0) (type default))
   )
@@
     (stroke (width 0) (type default))
   )
+  (wire (pts (xy 61.976 327.152) (xy 61.976 328.168))
+    (stroke (width 0) (type default))
+  )
