File: 2206Q/riscduino_board/Riscduino_Debug_Rev1.0/Riscduino_Debug.kicad_pcb (KiCad board)
At the start: 2 copper layers, 70.6 x 53.7 mm, 86 parts, among them J1 Conn_01x06_Pin, J10 USB_B_Micro, J11 Conn_01x10_Pin, J2 Conn_01x08_Pin, J3 Conn_01x01, J4 Conn_02x04_Odd_Even, J5 ISP, J6 Conn_01x01, J7 Conn_01x01, J8 Conn_01x01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

Commit message: BOM Added
Parts:
- C11, C2, C4, C5: value 0.1uf -> 0.1uF
- R22, R23, R24: value 0 Ohm -> 0E
Changed lines of the file:
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@@
         (effects (font (size 1.016 1.016) (thickness 0.1524)))
     )
-    (fp_text value "0.1uf" (at 0 1.43 90) (layer "F.Fab") hide
+    (fp_text value "0.1uF" (at 0 1.43 90) (layer "F.Fab") hide
         (effects (font (size 1 1) (thickness 0.15)))
     )
@@
         (effects (font (size 1.016 1.016) (thickness 0.1524)))
     )
-    (fp_text value "0.1uf" (at 0 1.43) (layer "F.Fab") hide
+    (fp_text value "0.1uF" (at 0 1.43) (layer "F.Fab") hide
         (effects (font (size 1 1) (thickness 0.15)))
     )
@@
         (effects (font (size 1.016 1.016) (thickness 0.1524)))
     )
-    (fp_text value "0.1uf" (at 0 1.43 90) (layer "F.Fab") hide
+    (fp_text value "0.1uF" (at 0 1.43 90) (layer "F.Fab") hide
         (effects (font (size 1 1) (thickness 0.15)))
     )
@@
         (effects (font (size 1.016 1.016) (thickness 0.1524)))
     )
-    (fp_text value "0.1uf" (at 0.254 1.27) (layer "F.Fab") hide
+    (fp_text value "0.1uF" (at 0.254 1.27) (layer "F.Fab") hide
         (effects (font (size 1 1) (thickness 0.15)))
     )
@@
         (effects (font (size 1.016 1.016) (thickness 0.1524)) (justify mirror))
     )
-    (fp_text value "0 Ohm" (at 0 -1.43 -270) (layer "B.Fab") hide
+    (fp_text value "0E" (at 0 -1.43 -270) (layer "B.Fab") hide
         (effects (font (size 1 1) (thickness 0.15)) (justify mirror))
     )
@@
         (effects (font (size 1.016 1.016) (thickness 0.1524)) (justify mirror))
     )
-    (fp_text value "0 Ohm" (at 0 -1.43 90) (layer "B.Fab") hide
+    (fp_text value "0E" (at 0 -1.43 90) (layer "B.Fab") hide
         (effects (font (size 1 1) (thickness 0.15)) (justify mirror))
     )
@@
         (effects (font (size 1.016 1.016) (thickness 0.1524)) (justify mirror))
     )
-    (fp_text value "0 Ohm" (at 0 -1.43) (layer "B.Fab") hide
+    (fp_text value "0E" (at 0 -1.43) (layer "B.Fab") hide
         (effects (font (size 1 1) (thickness 0.15)) (justify mirror))
     )
