File: 2206Q/riscduino_board/Riscduino_Debug_Rev1.0/Riscduino_Debug.kicad_sch (KiCad schematic)
At the start: 86 parts, among them J1 Conn_01x06_Pin, J10 USB_B_Micro, J11 Conn_01x10_Pin, J2 Conn_01x08_Pin, J3 Conn_01x01, J4 Conn_02x04_Odd_Even, J5 ISP, J6 Conn_01x01, J7 Conn_01x01, J8 Conn_01x01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

Commit message: BOM Added
Parts:
- C11, C2, C4, C5: value 0.1uf -> 0.1uF
- R22, R23, R24: value 0 Ohm -> 0E
Changed lines of the file:
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@@
   (symbol (lib_id "Device:R") (at 82.296 93.472 90) (unit 1)
     (in_bom yes) (on_board yes) (dnp no) (fields_autoplaced)
-    (property "Reference" "R23" (at 82.296 89.154 90)
+    (property "Reference" "R23" (at 82.296 88.9 90)
       (effects (font (size 1.27 1.27)))
     )
-    (property "Value" "0 Ohm" (at 82.296 91.694 90)
+    (property "Value" "0E" (at 82.296 91.44 90)
       (effects (font (size 1.27 1.27)))
     )
@@
   (symbol (lib_id "Device:C") (at 354.584 37.084 90) (unit 1)
     (in_bom yes) (on_board yes) (dnp no) (fields_autoplaced)
-    (property "Reference" "C11" (at 354.584 30.988 90)
+    (property "Reference" "C11" (at 354.584 30.48 90)
       (effects (font (size 1.27 1.27)))
     )
-    (property "Value" "0.1uf" (at 354.584 33.528 90)
+    (property "Value" "0.1uF" (at 354.584 33.02 90)
       (effects (font (size 1.27 1.27)))
     )
@@
   (symbol (lib_id "Device:C") (at 398.78 255.27 90) (unit 1)
     (in_bom yes) (on_board yes) (dnp no) (fields_autoplaced)
-    (property "Reference" "C4" (at 398.78 249.174 90)
+    (property "Reference" "C4" (at 398.78 248.92 90)
       (effects (font (size 1.27 1.27)))
     )
-    (property "Value" "0.1uf" (at 398.78 251.714 90)
+    (property "Value" "0.1uF" (at 398.78 251.46 90)
       (effects (font (size 1.27 1.27)))
     )
@@
   (symbol (lib_id "Device:C") (at 353.822 173.228 90) (unit 1)
     (in_bom yes) (on_board yes) (dnp no) (fields_autoplaced)
-    (property "Reference" "C5" (at 353.822 167.132 90)
+    (property "Reference" "C5" (at 353.822 167.64 90)
       (effects (font (size 1.27 1.27)))
     )
-    (property "Value" "0.1uf" (at 353.822 169.672 90)
+    (property "Value" "0.1uF" (at 353.822 170.18 90)
       (effects (font (size 1.27 1.27)))
     )
@@
       (effects (font (size 1.27 1.27)))
     )
-    (property "Value" "0 Ohm" (at 87.63 130.81 90)
+    (property "Value" "0E" (at 87.63 130.81 90)
       (effects (font (size 1.27 1.27)))
     )
@@
   (symbol (lib_id "Device:R") (at 169.418 120.65 90) (unit 1)
     (in_bom yes) (on_board yes) (dnp no) (fields_autoplaced)
-    (property "Reference" "R22" (at 169.418 116.332 90)
+    (property "Reference" "R22" (at 169.418 115.57 90)
       (effects (font (size 1.27 1.27)))
     )
-    (property "Value" "0 Ohm" (at 169.418 118.872 90)
+    (property "Value" "0E" (at 169.418 118.11 90)
       (effects (font (size 1.27 1.27)))
     )
@@
       (effects (font (size 1.27 1.27)))
     )
-    (property "Value" "0.1uf" (at 354.584 100.33 90)
+    (property "Value" "0.1uF" (at 354.584 100.33 90)
       (effects (font (size 1.27 1.27)))
     )
